File: Hardware/FilaClaceholder/fc.kicad_pcb (KiCad board)
At the start: 2 copper layers, 27.9 x 15.2 mm, 3 parts, among them J1 Conn_1, J2 Conn_2

Commit message: updated packages
Parts:
- H1: footprint MountingHole:MountingHole_3.2mm_M3_Pad_Via -> MountingHole:MountingHole_2.2mm_M2_Pad
- J1, J2: footprint Connector_PinSocket_2.54mm:PinSocket_2x04_P2.54mm_Vertical -> Connector_PinHeader_2.54mm:PinHeader_2x04_P2.54mm_Vertical
- moved H1 2.84 mm to (101.6, 48.3)
- moved J1 2.54 mm to (92.7, 44.5)
- moved J2 2.54 mm to (105.4, 49.5)
Connections:
- J1 pad 1: GND -> Net-(J1-Pad1)
- J1 pad 2: Net-(J1-Pad2) -> GND
- J1 pad 7: Net-(J1-Pad7) -> GND
- J1 pad 8: GND -> Net-(J1-Pad8)
- J2 pad 1: GND -> Net-(J2-Pad1)
- J2 pad 2: Net-(J2-Pad2) -> GND
- J2 pad 7: Net-(J2-Pad7) -> GND
- J2 pad 8: GND -> Net-(J2-Pad8)
Routing:
- net GND: vias 0 -> 4
Other:
- board size 27.9 x 15.2 mm -> 30.5 x 15.2 mm
- rule pad_to_mask_clearance: 0.051 -> 0
- board text added: "Fila Connector NULL v0.2 Sandbox Workshop 2021-04 Designed by Caorx Wangyw"
- board text added: "GND ONLY"
- board text added: "JLCJLCJLCJLC"
- board text removed: "Fila Placeholder v0.1 Sandbox Workshop Designed by Caorx Wangyw"
