File: Hardware/FilaDock/fc.kicad_pcb (KiCad board)
At the start: 2 copper layers, 30.5 x 15.2 mm, 4 parts, among them J1 Conn_1, J2 Conn_2, J3 PWR_IN, SW1 PowerSel

Commit message: Update
Parts:
- removed SW1: PowerSel, Button_Switch_SMD:SW_DIP_SPSTx02_Slide_KingTek_DSHP02TS_W7.62mm_P1.27mm
- added JP1: SolderJumper_3_Open, Jumper:SolderJumper-3_P1.3mm_Open_RoundedPad1.0x1.5mm, F.Cu at (109.2, 41.9)
Routing:
- net /5v_CON1: track 23.6 -> 16.6 mm
- net /5v_PWR: track 28.3 -> 31.8 mm, vias 2 -> 0
- net /5v_CON2: track 3.18 -> 6.12 mm
- net GND: vias 9 -> 3
Other:
- board text added: "Fila Dock v0.4 Sandbox 2021/9/12 By Caorx Wangyw"
- board text added: "PWR ONLY"
- board text removed: "Fila Dock v0.3 Sandbox 2021-04 By Caorx Wangyw"
